File: test_10/test_10/test_10.sch (KiCad schematic (older format))
At the start: 184 parts, among them J2 Array set 0

Commit message: renumber
Parts:
- renumbered H11 to H10, H12 to H11, H13 to H12, H8 to H7, H9 to H8, H10 to H9, J2 to J1, LS49 to LS10, LS21 to LS11, LS22 to LS12, LS23 to LS13, LS24 to LS14, LS25 to LS15, LS26 to LS16, LS27 to LS17, LS28 to LS18, LS50 to LS19, LS30 to LS20, LS11 to LS21, LS12 to LS22, LS13 to LS23, LS14 to LS24, LS15 to LS25, LS16 to LS26, LS17 to LS27, LS18 to LS28, LS19 to LS29, LS20 to LS30, LS41 to LS31, LS80 to LS32, LS47 to LS37, LS48 to LS38, LS51 to LS41, LS52 to LS42, LS53 to LS43, LS54 to LS44, LS55 to LS45, LS56 to LS46, LS57 to LS47, LS58 to LS48, LS59 to LS49, LS60 to LS50, LS71 to LS51, LS72 to LS52, LS73 to LS53, LS74 to LS54, LS75 to LS55, LS79 to LS56, LS78 to LS57, R3 to R1, R12 to R10, R120 to R100, R141 to R101, R142 to R102, R143 to R103, R144 to R104, R145 to R105, R146 to R106, R147 to R107, R151 to R108, R152 to R109, R23 to R11, R153 to R110, R154 to R111, R155 to R112, R156 to R113, R157 to R114, R24 to R12, R25 to R13, R26 to R14, R27 to R15, R28 to R16, R29 to R17, R30 to R18, R31 to R19, R4 to R2, R32 to R20, R43 to R21, R44 to R22, R45 to R23, R46 to R24, R47 to R25, R48 to R26, R49 to R27, R50 to R28, R51 to R29, R5 to R3, R52 to R30, R63 to R31, R64 to R32, R65 to R33, R66 to R34, R67 to R35, R68 to R36, R69 to R37, R70 to R38, R71 to R39, R6 to R4, R72 to R40, R1 to R41, R2 to R42, R13 to R43, R14 to R44, R15 to R45, R16 to R46, R17 to R47, R18 to R48, R19 to R49, R7 to R5, R20 to R50, R21 to R51, R22 to R52, R33 to R53, R34 to R54, R35 to R55, R36 to R56, R37 to R57, R38 to R58, R39 to R59, R8 to R6, R40 to R60, R41 to R61, R42 to R62, R53 to R63, R54 to R64, R55 to R65, R56 to R66, R57 to R67, R58 to R68, R59 to R69, R9 to R7, R60 to R70, R61 to R71, R62 to R72, R10 to R8, R101 to R81, R102 to R82, R103 to R83, R104 to R84, R105 to R85, R106 to R86, R107 to R87, R108 to R88, R109 to R89, R11 to R9, R110 to R90, R111 to R91, R112 to R92, R113 to R93, R114 to R94, R115 to R95, R116 to R96, R117 to R97, R118 to R98, R119 to R99

Commit message: pcb finish
Parts:
- added D1: LED, temp_pcb_lib:CREE_CXB1512, symbol Device:LED
- added J2: Array set 0, Connector_Phoenix_MC:PhoenixContact_MCV_1,5_2-G-3.5_1x02_P3.50mm_Vertical, symbol Connector_Generic:Conn_01x02
- added LS58, LS59: Ultrasonic, temp_pcb_lib:Buzzer_MSO-A1040H07T_D10mm_H7mm, symbol Device:Speaker_Ultrasound
- added R115, R116, R117, R118: 0.1Ω, Resistor_SMD:R_0603_1608Metric, symbol Device:R
Connections:
- net at J1.1 (Pin_1), R100.2, R108.2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: now also R116.2, R118.2; no longer J1.2 (Pin_2), R1.2, R10.2, R101.2, R102.2, R103.2, R104.2, R105.2, R106.2, R107.2, R2.2, R21.2, R22.2, R23.2, R24.2, R25.2, R26.2, R27.2, R28.2, R29.2, R3.2, R30.2, R4.2, R41.2, R42.2, R43.2, R44.2, R45.2, R46.2, R47.2, R48.2, R49.2, R5.2, R50.2, R6.2, R61.2, R62.2, R63.2, R64.2, R65.2, R66.2, R67.2, R68.2, R69.2, R7.2, R70.2, R8.2, R81.2, R82.2, R83.2, R84.2, R85.2, R86.2, R87.2, R88.2, R89.2, R9.2, R90.2
- new net: J1.2 (Pin_2), R1.2, R10.2, R101.2, R102.2, R103.2, R104.2, R105.2, R106.2, R107.2, R115.2, R117.2, R2.2, R21.2, R22.2, R23.2, R24.2, R25.2, R26.2, R27.2, R28.2, R29.2, R3.2, R30.2, R4.2, R41.2, R42.2, R43.2, R44.2, R45.2, R46.2, R47.2, R48.2, R49.2, R5.2, R50.2, R6.2, R61.2, R62.2, R63.2, R64.2, R65.2, R66.2, R67.2, R68.2, R69.2, R7.2, R70.2, R8.2, R81.2, R82.2, R83.2, R84.2, R85.2, R86.2, R87.2, R88.2, R89.2, R9.2, R90.2
- new net: LS58.1, R115.1
- new net: LS58.2, R116.1
- new net: LS59.1, R117.1
- new net: LS59.2, R118.1
- new net: D1.1 (K), J2.1 (Pin_1)
- new net: D1.2 (A), J2.2 (Pin_2)
Other:
- moved on the sheet: H1, H10, H11, H12, H2, H3, H4, H5, H6, H7, H8, H9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

Commit message: 3 trans mas
Parts:
- added LS60, LS61, LS62: Ultrasonic, temp_pcb_lib:Buzzer_MSO-A1040H07T_D10mm_H7mm, symbol Device:Speaker_Ultrasound
- added R119, R120, R121, R122, R123, R124: 0.1Ω, Resistor_SMD:R_0603_1608Metric, symbol Device:R
Connections:
- net at J1.1 (Pin_1), R100.2, R108.2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: now also R122.2, R123.2, R124.2
- net at J1.2 (Pin_2), R1.2, R10.2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: now also R119.2, R120.2, R121.2
- new net: LS60.1, R119.1
- new net: LS60.2, R122.1
- new net: LS61.1, R120.1
- new net: LS61.2, R123.1
- new net: LS62.1, R121.1
- new net: LS62.2, R124.1
Other:
- moved on the sheet: D1, J2
Changed lines of the file:
@@
 L Device:LED D1
 U 1 1 60F8A406
-P 9500 900
-F 0 "D1" H 9493 1117 50  0000 C CNN
-F 1 "LED" H 9493 1026 50  0000 C CNN
-F 2 "temp_pcb_lib:CREE_CXB1512" H 9500 900 50  0001 C CNN
-F 3 "~" H 9500 900 50  0001 C CNN
-	1    9500 900
+P 9550 3650
+F 0 "D1" H 9543 3867 50  0000 C CNN
+F 1 "LED" H 9543 3776 50  0000 C CNN
+F 2 "temp_pcb_lib:CREE_CXB1512" H 9550 3650 50  0001 C CNN
+F 3 "~" H 9550 3650 50  0001 C CNN
+	1    9550 3650
 	1    0    0    -1
 $EndComp
@@
 L Connector_Generic:Conn_01x02 J2
 U 1 1 6107F170
-P 8950 900
-F 0 "J2" H 8868 575 50  0000 C CNN
-F 1 "Array set 0" H 8868 666 50  0000 C CNN
-F 2 "Connector_Phoenix_MC:PhoenixContact_MCV_1,5_2-G-3.5_1x02_P3.50mm_Vertical" H 8950 900 50  0001 C CNN
-F 3 "~" H 8950 900 50  0001 C CNN
-	1    8950 900
+P 9000 3650
+F 0 "J2" H 8918 3325 50  0000 C CNN
+F 1 "Array set 0" H 8918 3416 50  0000 C CNN
+F 2 "Connector_Phoenix_MC:PhoenixContact_MCV_1,5_2-G-3.5_1x02_P3.50mm_Vertical" H 9000 3650 50  0001 C CNN
+F 3 "~" H 9000 3650 50  0001 C CNN
+	1    9000 3650
 	-1   0    0    -1
 $EndComp
 Wire Wire Line
-	9150 900  9350 900
+	9200 3650 9400 3650
 Wire Wire Line
-	9150 1000 9650 1000
+	9200 3750 9700 3750
 Wire Wire Line
-	9650 1000 9650 900
+	9700 3750 9700 3650
 Wire Wire Line
 	3400 750  3400 1000
 Wire Wire Line
 	2300 850  3500 850
+$Comp
+L Device:Speaker_Ultrasound LS60
+U 1 1 610B34BB
+P 9050 1000
+F 0 "LS60" H 8950 700 50  0000 L CNN
+F 1 "Ultrasonic" H 8950 600 50  0000 L CNN
+F 2 "temp_pcb_lib:Buzzer_MSO-A1040H07T_D10mm_H7mm" H 9015 950 50  0001 C CNN
+F 3 "~" H 9015 950 50  0001 C CNN
+	1    9050 1000
+	1    0    0    -1
+$EndComp
+Wire Wire Line
+	8850 1000 8700 1000
+$Comp
+L Device:Speaker_Ultrasound LS61
+U 1 1 610B34E0
+P 9050 1650
+F 0 "LS61" H 8950 1350 50  0000 L CNN
+F 1 "Ultrasonic" H 8950 1250 50  0000 L CNN
+F 2 "temp_pcb_lib:Buzzer_MSO-A1040H07T_D10mm_H7mm" H 9015 1600 50  0001 C CNN
+F 3 "~" H 9015 1600 50  0001 C CNN
+	1    9050 1650
+	1    0    0    -1
+$EndComp
+Wire Wire Line
+	8850 1650 8700 1650
+Wire Wire Line
+	8850 1750 8750 1750
+$Comp
+L Device:Speaker_Ultrasound LS62
+U 1 1 610B34EC
+P 9050 2300
+F 0 "LS62" H 8950 2000 50  0000 L CNN
+F 1 "Ultrasonic" H 8950 1900 50  0000 L CNN
+F 2 "temp_pcb_lib:Buzzer_MSO-A1040H07T_D10mm_H7mm" H 9015 2250 50  0001 C CNN
+F 3 "~" H 9015 2250 50  0001 C CNN
+	1    9050 2300
+	1    0    0    -1
+$EndComp
+Wire Wire Line
+	8850 2300 8700 2300
+Wire Wire Line
+	8850 2400 8750 2400
+$Comp
+L Device:R R119
+U 1 1 610B34F8
+P 8550 1000
+F 0 "R119" V 8450 850 50  0000 C CNN
+F 1 "0.1Ω" V 8450 1100 50  0000 C CNN
+F 2 "Resistor_SMD:R_0603_1608Metric" V 8480 1000 50  0001 C CNN
+F 3 "~" H 8550 1000 50  0001 C CNN
+	1    8550 1000
+	0    1    1    0
+$EndComp
+Wire Wire Line
+	8400 1000 8200 1000
+Wire Wire Line
+	8850 1100 8750 1100
+$Comp
+L Device:R R122
+U 1 1 610B3504
+P 8600 1100
+F 0 "R122" V 8700 950 50  0000 C CNN
+F 1 "0.1Ω" V 8700 1250 50  0000 C CNN
+F 2 "Resistor_SMD:R_0603_1608Metric" V 8530 1100 50  0001 C CNN
+F 3 "~" H 8600 1100 50  0001 C CNN
+	1    8600 1100
+	0    1    1    0
+$EndComp
+Wire Wire Line
+	8450 1100 8300 1100
+$Comp
+L Device:R R120
+U 1 1 610B350F
+P 8550 1650
+F 0 "R120" V 8450 1500 50  0000 C CNN
+F 1 "0.1Ω" V 8450 1750 50  0000 C CNN
+F 2 "Resistor_SMD:R_0603_1608Metric" V 8480 1650 50  0001 C CNN
+F 3 "~" H 8550 1650 50  0001 C CNN
+	1    8550 1650
+	0    1    1    0
+$EndComp
+$Comp
+L Device:R R123
+U 1 1 610B3519
+P 8600 1750
+F 0 "R123" V 8700 1600 50  0000 C CNN
+F 1 "0.1Ω" V 8700 1900 50  0000 C CNN
+F 2 "Resistor_SMD:R_0603_1608Metric" V 8530 1750 50  0001 C CNN
+F 3 "~" H 8600 1750 50  0001 C CNN
+	1    8600 1750
+	0    1    1    0
+$EndComp
+Wire Wire Line
+	8400 1650 8200 1650
+Wire Wire Line
+	8450 1750 8300 1750
+$Comp
+L Device:R R121
+U 1 1 610B3525
+P 8550 2300
+F 0 "R121" V 8450 2150 50  0000 C CNN
+F 1 "0.1Ω" V 8450 2400 50  0000 C CNN
+F 2 "Resistor_SMD:R_0603_1608Metric" V 8480 2300 50  0001 C CNN
+F 3 "~" H 8550 2300 50  0001 C CNN
+	1    8550 2300
+	0    1    1    0
+$EndComp
+$Comp
+L Device:R R124
+U 1 1 610B352F
+P 8600 2400
+F 0 "R124" V 8700 2250 50  0000 C CNN
+F 1 "0.1Ω" V 8700 2550 50  0000 C CNN
+F 2 "Resistor_SMD:R_0603_1608Metric" V 8530 2400 50  0001 C CNN
+F 3 "~" H 8600 2400 50  0001 C CNN
+	1    8600 2400
+	0    1    1    0
+$EndComp
+Wire Wire Line
+	8450 2400 8300 2400
+Wire Wire Line
+	8400 2300 8200 2300
+Wire Wire Line
+	7000 750  8200 750
+Wire Wire Line
+	8200 750  8200 1000
+Connection ~ 7000 750
+Connection ~ 8200 1000
+Wire Wire Line
+	8200 1000 8200 1650
+Connection ~ 8200 1650
+Wire Wire Line
+	8200 1650 8200 2300
+Wire Wire Line
+	8300 2400 8300 1750
+Wire Wire Line
+	8300 850  7100 850
+Connection ~ 8300 1100
+Wire Wire Line
+	8300 1100 8300 850
+Connection ~ 8300 1750
+Wire Wire Line
+	8300 1750 8300 1100
+Connection ~ 7100 850
 $EndSCHEMATC

Commit message: 3 trans mas
Parts:
- renumbered R115 to R108, R117 to R109, R108 to R110, R109 to R111, R110 to R112, R111 to R113, R112 to R114, R113 to R115, R114 to R116, R116 to R117
Changed lines of the file:
@@
 	7650 1100 7550 1100
 $Comp
-L Device:R R108
+L Device:R R110
 U 1 1 60BD97ED
 P 7400 1100
-F 0 "R108" V 7500 950 50  0000 C CNN
+F 0 "R110" V 7500 950 50  0000 C CNN
 F 1 "0.1Ω" V 7500 1250 50  0000 C CNN
 F 2 "Resistor_SMD:R_0603_1608Metric" V 7330 1100 50  0001 C CNN
@@
 $EndComp
 $Comp
-L Device:R R109
+L Device:R R111
 U 1 1 60BD9802
 P 7400 1750
-F 0 "R109" V 7500 1600 50  0000 C CNN
+F 0 "R111" V 7500 1600 50  0000 C CNN
 F 1 "0.1Ω" V 7500 1900 50  0000 C CNN
 F 2 "Resistor_SMD:R_0603_1608Metric" V 7330 1750 50  0001 C CNN
@@
 $EndComp
 $Comp
-L Device:R R110
+L Device:R R112
 U 1 1 60BD9818
 P 7400 2400
-F 0 "R110" V 7500 2250 50  0000 C CNN
+F 0 "R112" V 7500 2250 50  0000 C CNN
 F 1 "0.1Ω" V 7500 2550 50  0000 C CNN
 F 2 "Resistor_SMD:R_0603_1608Metric" V 7330 2400 50  0001 C CNN
@@
 $EndComp
 $Comp
-L Device:R R111
+L Device:R R113
 U 1 1 60BD982C
 P 7400 3050
-F 0 "R111" V 7500 2900 50  0000 C CNN
+F 0 "R113" V 7500 2900 50  0000 C CNN
 F 1 "0.1Ω" V 7500 3200 50  0000 C CNN
 F 2 "Resistor_SMD:R_0603_1608Metric" V 7330 3050 50  0001 C CNN
@@
 $EndComp
 $Comp
-L Device:R R112
+L Device:R R114
 U 1 1 60BD9840
 P 7400 3700
-F 0 "R112" V 7500 3550 50  0000 C CNN
+F 0 "R114" V 7500 3550 50  0000 C CNN
 F 1 "0.1Ω" V 7500 3850 50  0000 C CNN
 F 2 "Resistor_SMD:R_0603_1608Metric" V 7330 3700 50  0001 C CNN
@@
 $EndComp
 $Comp
-L Device:R R113
+L Device:R R115
 U 1 1 60BD9854
 P 7400 4350
-F 0 "R113" V 7500 4200 50  0000 C CNN
+F 0 "R115" V 7500 4200 50  0000 C CNN
 F 1 "0.1Ω" V 7500 4500 50  0000 C CNN
 F 2 "Resistor_SMD:R_0603_1608Metric" V 7330 4350 50  0001 C CNN
@@
 $EndComp
 $Comp
-L Device:R R114
+L Device:R R116
 U 1 1 60BD9868
 P 7400 4950
-F 0 "R114" V 7500 4800 50  0000 C CNN
+F 0 "R116" V 7500 4800 50  0000 C CNN
 F 1 "0.1Ω" V 7500 5100 50  0000 C CNN
 F 2 "Resistor_SMD:R_0603_1608Metric" V 7330 4950 50  0001 C CNN
@@
 	7000 4850 7000 5450
 $Comp
-L Device:R R115
+L Device:R R108
 U 1 1 60F2870D
 P 7350 5450
-F 0 "R115" V 7250 5300 50  0000 C CNN
+F 0 "R108" V 7250 5300 50  0000 C CNN
 F 1 "0.1Ω" V 7250 5550 50  0000 C CNN
 F 2 "Resistor_SMD:R_0603_1608Metric" V 7280 5450 50  0001 C CNN
@@
 $EndComp
 $Comp
-L Device:R R116
+L Device:R R117
 U 1 1 60F28717
 P 7400 5550
-F 0 "R116" V 7500 5400 50  0000 C CNN
+F 0 "R117" V 7500 5400 50  0000 C CNN
 F 1 "0.1Ω" V 7500 5700 50  0000 C CNN
 F 2 "Resistor_SMD:R_0603_1608Metric" V 7330 5550 50  0001 C CNN
@@
 	7000 5450 7000 6050
 $Comp
-L Device:R R117
+L Device:R R109
 U 1 1 60F4CE6E
 P 7350 6050
-F 0 "R117" V 7250 5900 50  0000 C CNN
+F 0 "R109" V 7250 5900 50  0000 C CNN
 F 1 "0.1Ω" V 7250 6150 50  0000 C CNN
 F 2 "Resistor_SMD:R_0603_1608Metric" V 7280 6050 50  0001 C CNN
